File: viper/_autosave-viper.kicad_sch (KiCad schematic)
At the start: 57 parts, among them J1 Barrel_Jack, J10 DEBUG PINS, J11 Conn_01x05_Male, J12 Pimoroni Inky pHAT, J13 Pimoroni BLINKT!, J2 Raspberry Pi Zero W2, J3 Raspberry Pi Zero W2, J4 Adafruit CharliePlex Bonnet, J5 Adafruit CharliePlex Bonnet, J6 Pimoroni Inky pHAT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

Commit message: feat: switches
Signed-off-by: Matt Gleich <git@mattglei.ch>
Parts:
- gave numbers to parts that had none: 12
