File: viper/_autosave-viper.kicad_pcb (KiCad board)
At the start: 2 copper layers, 258.2 x 197 mm, 58 parts, among them J1 Barrel_Jack, J10 DEBUG PINS, J11 Conn_01x05_Male, J12 Pimoroni Inky pHAT, J13 Pimoroni BLINKT!, J14 DEBUG Pins, J15 Adafruit Charlieplex Bonnet, J2 Raspberry Pi Zero W2, J3 Raspberry Pi Zero W2, J4 Adafruit CharliePlex Bonnet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

Commit message: feat: mark ii routing
Signed-off-by: Matt Gleich <git@mattglei.ch>
Routing:
- net VBUS: track 1040.7 -> 1117.9 mm
- net GND: track 1029.9 -> 1105.8 mm, vias 26 -> 28
- net /RESET: track 180.6 -> 188.9 mm
- net /3.3V: track 183.3 -> 184.3 mm
- net /BUSY: track 185.9 -> 186.8 mm
- net /SCL 01: track 181.1 -> 182.1 mm
- net /SDA 03: track 113.7 -> 114.6 mm
- net /SDA 01: track 179.1 -> 180.1 mm
