File: viper/viper.kicad_pcb (KiCad board)
At the start: 2 copper layers, 258.2 x 197 mm, 58 parts, among them J1 Barrel_Jack, J10 DEBUG PINS, J11 Conn_01x05_Male, J12 Pimoroni Inky pHAT, J13 Pimoroni BLINKT!, J14 DEBUG Pins, J15 Adafruit Charlieplex Bonnet, J2 Raspberry Pi Zero W2, J3 Raspberry Pi Zero W2, J4 Adafruit CharliePlex Bonnet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

Commit message: feat: graphics
Signed-off-by: Matt Gleich <git@mattglei.ch>
Parts:
- added G***: LOGO, Viper:logo_mask, F.Cu at (258.8, 63.2)
- added G***: LOGO, Viper:mark_II, F.Cu at (257.0, 92.5)
- added G***: LOGO, Viper:logo_copper, F.Cu at (258.8, 63.2)
- added G***: LOGO, Viper:mark_I, F.Cu at (136.4, 91.9)
- moved Brd2 107.4 mm to (351.4, 158.2)
- moved Brd1 72.9 mm to (72.7, 252.5)
- moved U2 72.9 mm to (43.9, 250.6)
- moved U3 71.7 mm to (97.3, 207.8)
- moved J12 4.20 mm to (151.8, 106.8)
- moved J13 4.20 mm to (184.7, 106.8)
- moved J6 4.20 mm to (239.7, 154.2)
- moved J9 4.20 mm to (206.8, 154.2)
- moved J2 4.20 mm to (109.5, 154.1)
- moved J4 4.20 mm to (119.0, 106.6)
- moved J3 4.20 mm to (281.9, 106.0)
- moved J5 4.20 mm to (272.3, 154.2)
Routing:
- net VBUS: track 1040.7 -> 1126.2 mm
- net GND: track 1029.9 -> 1109.5 mm, vias 26 -> 28
- net /RESET: track 180.6 -> 188.9 mm
- net /3.3V: track 183.3 -> 184.3 mm
- net /SCL 01: track 181.1 -> 182.1 mm
- net /SDA 03: track 113.7 -> 114.6 mm
- net /BUSY: track 185.9 -> 186.8 mm
- net /SDA 01: track 179.1 -> 180.1 mm
Other:
- board size 258.2 x 197 mm -> 238.8 x 197 mm

Commit message: feat: final connections
Signed-off-by: Matt Gleich <git@mattglei.ch>
Parts:
- removed Brd2, Brd3: SSD1306, SSD1306:128x64OLED
- removed D12, D14: LED, LED_THT:LED_D5.0mm
- removed J8: DEBUG PINS, Connector_PinHeader_2.54mm:PinHeader_2x02_P2.54mm_Vertical
- removed R13, R14: 330Ω, Resistor_THT:R_Axial_DIN0309_L9.0mm_D3.2mm_P12.70mm_Horizontal
- removed S8: MARK VI, M2012SA1W03:M2012SA1W03
- removed U3: Pico, Pico:RPi_Pico_SMD_TH
- added G***: LOGO, Viper:mark_V, F.Cu at (293.6, 215.0)
- added G***: LOGO, Viper:mark_V, F.Cu at (222.5, 225.7)
- added G***: LOGO, Viper:mark_III, F.Cu at (293.6, 196.2)
- added G***: LOGO, Viper:mark_IV, F.Cu at (154.8, 226.3)
- added G***: LOGO, Viper:mark_III, F.Cu at (124.8, 178.6)
- added G***: LOGO, Viper:mark_I, F.Cu at (293.6, 177.4)
- added G***: LOGO, Viper:mark_II, F.Cu at (293.6, 187.0)
- added G***: LOGO, Viper:mark_IV, F.Cu at (293.6, 205.4)
- moved U4 222.4 mm to (158.9, 195.5), turned to 180 degrees
- moved J15 220.5 mm to (205.7, 223.4), turned to 180 degrees
- moved J7 198.1 mm to (111.1, 221.4)
- moved S7 194.6 mm to (255.0, 225.5), turned to 90 degrees
- moved Brd1 76.0 mm to (125.7, 198.0)
- moved U2 71.8 mm to (94.6, 199.8)
- moved J14 59.4 mm to (173.0, 228.0), turned to 180 degrees
- moved J10 58.2 mm to (239.7, 226.8), turned to 180 degrees
- moved J11 33.2 mm to (245.4, 188.3)
- moved U1 24.5 mm to (226.6, 193.9)
- moved G*** 8.44 mm to (250.4, 64.3) (x2)
Connections:
- Brd1 pad 1: Net-(Brd1-Pad1) -> GND
- J12 pad 1: /3.3V -> /1 3.3V
- J12 pad 11: /BUSY -> /1 BUSY
- J12 pad 13: /RESET -> /1 RESET
- J12 pad 15: /DATA -> /1 DATA
- J12 pad 19: /SPI0 MOSI -> /1 SPI0 MOSI
- J12 pad 23: /SPI0 SCLK -> /1 SPI0 SCLK
- J12 pad 24: /CS -> /1 CS
- J12 pad 3: /SDA 01 -> /1 SDA 01
- J12 pad 5: /SCL 01 -> /1 SCL 01
- J13 pad 16: /GPIO 23 -> /1 GPIO 23
- J13 pad 18: /GPIO 24 -> /1 GPIO 24
- J2 pad 1: /3.3V -> /1 3.3V
- J2 pad 11: /BUSY -> /1 BUSY
- J2 pad 13: /RESET -> /1 RESET
- J2 pad 15: /DATA -> /1 DATA
- J2 pad 16: /GPIO 23 -> /1 GPIO 23
- J2 pad 18: /GPIO 24 -> /1 GPIO 24
- J2 pad 19: /SPI0 MOSI -> /1 SPI0 MOSI
- J2 pad 23: /SPI0 SCLK -> /1 SPI0 SCLK
- J2 pad 24: /CS -> /1 CS
- J2 pad 29: /SCL 03 -> /1 SCL 03
- J2 pad 3: /SDA 01 -> /1 SDA 01
- J2 pad 5: /SCL 01 -> /1 SCL 01
- J2 pad 7: /SDA 03 -> /1 SDA 03
- J3 pad 1: /3.3V -> /2 3.3V
- J3 pad 11: /BUSY -> /2 BUSY
- J3 pad 13: /RESET -> /2 RESET
- J3 pad 15: /DATA -> /2 DATA
- J3 pad 16: /GPIO 23 -> /2 GPIO 23
- J3 pad 18: /GPIO 24 -> /2 GPIO 24
- J3 pad 19: /SPI0 MOSI -> /2 SPI0 MOSI
- J3 pad 23: /SPI0 SCLK -> /2 SPI0 SCLK
- J3 pad 24: /CS -> /2 CS
- J3 pad 29: /SCL 03 -> /2 SCL 03
- J3 pad 3: /SDA 01 -> /2 SDA 01
- J3 pad 5: /SCL 01 -> /2 SCL 01
- J3 pad 7: /SDA 03 -> /2 SDA 03
- J4 pad 1: /3.3V -> /1 3.3V
- J4 pad 3: /SDA 03 -> /1 SDA 03
- J4 pad 5: /SCL 03 -> /1 SCL 03
- J5 pad 1: /3.3V -> /2 3.3V
- J5 pad 3: /SDA 03 -> /2 SDA 03
- J5 pad 5: /SCL 03 -> /2 SCL 03
- J6 pad 1: /3.3V -> /2 3.3V
- J6 pad 11: /BUSY -> /2 BUSY
- J6 pad 13: /RESET -> /2 RESET
- J6 pad 15: /DATA -> /2 DATA
- J6 pad 19: /SPI0 MOSI -> /2 SPI0 MOSI
- J6 pad 23: /SPI0 SCLK -> /2 SPI0 SCLK
- J6 pad 24: /CS -> /2 CS
- J6 pad 3: /SDA 01 -> /2 SDA 01
- J6 pad 5: /SCL 01 -> /2 SCL 01
- J9 pad 16: /GPIO 23 -> /2 GPIO 23
- J9 pad 18: /GPIO 24 -> /2 GPIO 24
- U2 pad 38: Net-(Brd1-Pad1) -> unconnected-(U2-Pad38)
Routing:
- net VBUS: track 1126.2 -> 1766.5 mm, vias 2 -> 5
- net GND: track 1109.5 -> 1436.6 mm
- net /GPIO 24: track 284.9 -> 0.00 mm
- net /GPIO 23: track 266.1 -> 0.00 mm
- net /CS: track 228.9 -> 0.00 mm, vias 2 -> 0
- net /SPI0 SCLK: track 200.9 -> 0.00 mm, vias 2 -> 0
- net /SPI0 MOSI: track 198.5 -> 0.00 mm, vias 2 -> 0
- net /DATA: track 190.9 -> 0.00 mm, vias 2 -> 0
- net /RESET: track 188.9 -> 0.00 mm, vias 2 -> 0
- net /BUSY: track 186.8 -> 0.00 mm, vias 2 -> 0
- net /3.3V: track 184.3 -> 0.00 mm
- net /SCL 01: track 182.1 -> 0.00 mm, vias 2 -> 0
- net /SDA 01: track 180.1 -> 0.00 mm, vias 2 -> 0
- net /2 GPIO 24: track 0.00 -> 142.9 mm
- net /1 GPIO 24: track 0.00 -> 142.0 mm
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Other:
- board size 238.8 x 197 mm -> 238.8 x 193.7 mm
- board text removed: "MARK VI"

Commit message: feat: fixes
Signed-off-by: Matt Gleich <git@mattglei.ch>
Parts:
- removed the G*** at (293.6, 215.0)
- removed the G*** at (293.6, 196.2)
- removed the G*** at (293.6, 177.4)
- removed the G*** at (293.6, 187.0)
- removed the G*** at (293.6, 205.4)
- added G***: LOGO, Viper:marks, F.Cu at (305.2, 198.7)
- added G***: LOGO, Viper:back, F.Cu at (257.7, 64.3)
- J11: value Conn_01x05_Male -> Adafruit Quad Alphanumeric Display (I2C Backpack)
- moved J3 48.3 mm to (284.5, 154.2), turned to 180 degrees
- moved J2 46.4 mm to (106.9, 107.7), turned to 0 degrees
- moved J11 33.6 mm to (274.2, 170.9), turned to -90 degrees
Connections:
- U1 pad 39: unconnected-(U1-Pad39) -> VBUS
- U1 pad 40: VBUS -> unconnected-(U1-Pad40)
- U2 pad 39: unconnected-(U2-Pad39) -> VBUS
- U2 pad 40: VBUS -> unconnected-(U2-Pad40)
- U4 pad 39: unconnected-(U4-Pad39) -> VBUS
- U4 pad 40: VBUS -> unconnected-(U4-Pad40)
Routing:
- net VBUS: track 1766.5 -> 1877.2 mm
- net GND: track 1436.6 -> 1501.2 mm
- net /2 3.3V: track 92.6 -> 49.1 mm
- net /1 3.3V: track 91.6 -> 51.1 mm
- net /2 SCL 03: track 46.1 -> 85.0 mm
- net /1 SCL 03: track 45.1 -> 82.9 mm
- net Net-(J11-Pad3): track 35.8 -> 70.3 mm, vias 0 -> 3
- net /2 SDA 01: track 90.5 -> 57.5 mm
- net /1 SDA 01: track 89.6 -> 57.9 mm
- net Net-(J11-Pad1): track 41.1 -> 72.4 mm, vias 0 -> 3
- net Net-(J11-Pad2): track 36.4 -> 65.2 mm, vias 0 -> 3
- net /2 SCL 01: track 91.5 -> 63.2 mm
- net /1 SCL 01: track 90.6 -> 63.6 mm
- net /1 CS: track 113.9 -> 138.6 mm
- net /2 CS: track 115.0 -> 138.2 mm
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
Commit message: feat: final viper board changes
Signed-off-by: Matt Gleich <git@mattglei.ch>
Parts:
- J11: value Adafruit Quad Alphanumeric Display (I2C Backpack) -> Adafruit Quad Alphanumeric I2C Backpack
- moved J4 48.3 mm to (121.5, 154.9), turned to 180 degrees
- moved J15 48.3 mm to (203.2, 175.1), turned to 0 degrees
- moved J12 48.3 mm to (154.3, 155.1), turned to 180 degrees
- moved J13 48.1 mm to (187.2, 154.8), turned to 180 degrees
- moved J6 47.9 mm to (237.4, 106.4), turned to 0 degrees
- moved J5 47.8 mm to (270.1, 106.5), turned to 0 degrees
- moved J9 47.7 mm to (204.5, 106.6), turned to 0 degrees
- moved G*** 6.54 mm to (251.2, 65.2)
- moved J3 0.65 mm to (284.8, 153.7)
- moved G*** 0.51 mm to (257.0, 93.0)
Connections:
- J11 pad 3: Net-(J11-Pad3) -> GND
- J15 pad 6: Net-(J15-Pad6) -> GND
- U1 pad 3: GND -> unconnected-(U1-Pad3)
- U1 pad 38: Net-(J11-Pad3) -> GND
- U2 pad 3: GND -> unconnected-(U2-Pad3)
- U2 pad 38: unconnected-(U2-Pad38) -> GND
- U4 pad 3: GND -> unconnected-(U4-Pad3)
- U4 pad 38: Net-(J15-Pad6) -> GND
Routing:
- net VBUS: track 1877.2 -> 1578.7 mm
- net GND: track 1501.2 -> 1396.9 mm, vias 28 -> 31
- net /2 3.3V: track 49.1 -> 145.8 mm, vias 0 -> 1
- net /1 3.3V: track 51.1 -> 145.8 mm, vias 0 -> 1
- net Net-(J11-Pad3): track 70.3 -> 0.00 mm, vias 3 -> 0
- net Net-(J15-Pad6): track 54.8 -> 0.00 mm, vias 2 -> 0
- net /2 SDA 03: track 35.1 -> 86.0 mm
- net /1 SDA 03: track 35.4 -> 86.0 mm
- net /2 SDA 01: track 57.5 -> 97.8 mm
- net /1 SDA 01: track 57.9 -> 97.8 mm
- net /1 SCL 03: track 82.9 -> 122.6 mm
- net /2 SCL 03: track 85.0 -> 122.6 mm
- net /2 SCL 01: track 63.2 -> 100.4 mm
- net /1 SCL 01: track 63.6 -> 100.4 mm
- net Net-(J15-Pad5): track 80.6 -> 56.9 mm
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Other:
- board size 238.8 x 193.7 mm -> 239.5 x 193.7 mm
- board text added: "MARK I DATA BUS"
- board text added: "MARK II DATA BUS"
