File: viper/viper.kicad_sch (KiCad schematic)
At the start: 57 parts, among them J1 Barrel_Jack, J10 DEBUG PINS, J11 Conn_01x05_Male, J12 Pimoroni Inky pHAT, J13 Pimoroni BLINKT!, J14 DEBUG Pins, J15 Adafruit Charlieplex Bonnet, J2 Raspberry Pi Zero W2, J3 Raspberry Pi Zero W2, J4 Adafruit CharliePlex Bonnet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

Commit message: feat: final connections
Signed-off-by: Matt Gleich <git@mattglei.ch>
Parts:
- removed Brd2: SSD1306, SSD1306:128x64OLED, symbol SSD1306:SSD1306
- removed D12, D14: LED, LED_THT:LED_D5.0mm, symbol Device:LED
- removed J8: DEBUG PINS, Connector_PinHeader_2.54mm:PinHeader_2x02_P2.54mm_Vertical, symbol Connector_Generic:Conn_02x02_Counter_Clockwise
- removed R13, R14: 330Ω, Resistor_THT:R_Axial_DIN0309_L9.0mm_D3.2mm_P12.70mm_Horizontal, symbol Device:R_US
- removed S8: (no value), M2012SA1W03:M2012SA1W03, symbol M2012SA1W03:M2012SA1W03
- removed U3: Pico, Pico:RPi_Pico_SMD_TH, symbol MCU_RaspberryPi_and_Boards:Pico
Connections:
- net GND: now also Brd1.1 (GND)
- net at U2.38 (GND): no longer Brd1.1 (GND)
- net 3.3V renamed 1 3.3V
- net 1 3.3V: no longer J3.1 (Pin_1), J5.1 (Pin_1), J6.1 (Pin_1)
- net BUSY renamed 1 BUSY
- net 1 BUSY: no longer J3.11 (Pin_11), J6.11 (Pin_11)
- net CS renamed 1 CS
- net 1 CS: no longer J3.24 (Pin_24), J6.24 (Pin_24)
- net DATA renamed 1 DATA
- net 1 DATA: no longer J3.15 (Pin_15), J6.15 (Pin_15)
- net GPIO 23 renamed 1 GPIO 23
- net 1 GPIO 23: no longer J3.16 (Pin_16), J9.16 (Pin_16)
- net GPIO 24 renamed 1 GPIO 24
- net 1 GPIO 24: no longer J3.18 (Pin_18), J9.18 (Pin_18)
- net RESET renamed 1 RESET
- net 1 RESET: no longer J3.13 (Pin_13), J6.13 (Pin_13)
- net SCL 01 renamed 1 SCL 01
- net 1 SCL 01: no longer J3.5 (Pin_5), J6.5 (Pin_5)
- net SCL 03 renamed 1 SCL 03
- net 1 SCL 03: no longer J3.29 (Pin_29), J5.5 (Pin_5)
- net SDA 01 renamed 1 SDA 01
- net 1 SDA 01: no longer J3.3 (Pin_3), J6.3 (Pin_3)
- net SDA 03 renamed 1 SDA 03
- net 1 SDA 03: no longer J3.7 (Pin_7), J5.3 (Pin_3)
- net SPI0 MOSI renamed 1 SPI0 MOSI
- net 1 SPI0 MOSI: no longer J3.19 (Pin_19), J6.19 (Pin_19)
- net SPI0 SCLK renamed 1 SPI0 SCLK
- net 1 SPI0 SCLK: no longer J3.23 (Pin_23), J6.23 (Pin_23)
- new net 2 3.3V: J3.1 (Pin_1), J5.1 (Pin_1), J6.1 (Pin_1)
- new net 2 BUSY: J3.11 (Pin_11), J6.11 (Pin_11)
- new net 2 CS: J3.24 (Pin_24), J6.24 (Pin_24)
- new net 2 DATA: J3.15 (Pin_15), J6.15 (Pin_15)
- new net 2 GPIO 23: J3.16 (Pin_16), J9.16 (Pin_16)
- new net 2 GPIO 24: J3.18 (Pin_18), J9.18 (Pin_18)
- new net 2 RESET: J3.13 (Pin_13), J6.13 (Pin_13)
- new net 2 SCL 01: J3.5 (Pin_5), J6.5 (Pin_5)
- new net 2 SCL 03: J3.29 (Pin_29), J5.5 (Pin_5)
- new net 2 SDA 01: J3.3 (Pin_3), J6.3 (Pin_3)
- new net 2 SDA 03: J3.7 (Pin_7), J5.3 (Pin_3)
- new net 2 SPI0 MOSI: J3.19 (Pin_19), J6.19 (Pin_19)
- new net 2 SPI0 SCLK: J3.23 (Pin_23), J6.23 (Pin_23)
- no-connect marks 413 -> 382
Other:
- note removed: "MARK VI"

Commit message: feat: fixes
Signed-off-by: Matt Gleich <git@mattglei.ch>
Connections:
- net VBUS: now also U1.39 (VSYS), U2.39 (VSYS), U4.39 (VSYS); no longer U1.40 (VBUS), U2.40 (VBUS), U4.40 (VBUS)
Changed lines of the file:
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@@
   (junction (at 81.28 57.15) (diameter 0) (color 0 0 0 0)
   )
-  (junction (at 280.67 121.92) (diameter 0) (color 0 0 0 0)
-  )
   (junction (at 88.9 35.56) (diameter 0) (color 0 0 0 0)
   )
@@
   (junction (at 48.26 27.94) (diameter 0) (color 0 0 0 0)
   )
+  (junction (at 280.67 123.19) (diameter 0) (color 0 0 0 0)
+  )
   (no_connect (at 121.92 248.92))
   (no_connect (at 45.72 259.08))
@@
   (no_connect (at 33.02 156.21))
   (no_connect (at 332.74 165.1))
-  (no_connect (at 367.03 45.72))
   (no_connect (at 166.37 233.68))
   (no_connect (at 166.37 151.13))
@@
   (no_connect (at 332.74 144.78))
   (no_connect (at 379.73 85.09))
+  (no_connect (at 270.51 121.92))
   (no_connect (at 134.62 261.62))
   (no_connect (at 179.07 161.29))
@@
   (no_connect (at 331.47 60.96))
   (no_connect (at 367.03 71.12))
+  (no_connect (at 368.3 121.92))
   (no_connect (at 166.37 218.44))
   (no_connect (at 392.43 87.63))
@@
   (no_connect (at 179.07 256.54))
   (no_connect (at 33.02 161.29))
-  (no_connect (at 368.3 124.46))
   (no_connect (at 368.3 137.16))
   (no_connect (at 368.3 127))
@@
   (no_connect (at 332.74 154.94))
   (no_connect (at 90.17 226.06))
-  (no_connect (at 270.51 124.46))
   (no_connect (at 134.62 166.37))
   (no_connect (at 90.17 256.54))
@@
   (no_connect (at 121.92 179.07))
   (no_connect (at 77.47 256.54))
+  (no_connect (at 367.03 43.18))
   (no_connect (at 134.62 241.3))
   (no_connect (at 134.62 184.15))
@@
     (stroke (width 0) (type default) (color 0 0 0 0))
   )
-  (wire (pts (xy 270.51 121.92) (xy 280.67 121.92))
-    (stroke (width 0) (type default) (color 0 0 0 0))
-  )
   (bus (pts (xy 193.04 218.44) (xy 193.04 231.14))
     (stroke (width 0) (type default) (color 0 0 0 0))
@@
     (stroke (width 0) (type default) (color 0 0 0 0))
   )
-  (wire (pts (xy 368.3 121.92) (xy 378.46 121.92))
-    (stroke (width 0) (type default) (color 0 0 0 0))
-  )
   (bus (pts (xy 59.69 218.44) (xy 59.69 231.14))
     (stroke (width 0) (type default) (color 0 0 0 0))
@@
     (stroke (width 0) (type default) (color 0 0 0 0))
   )
+  (wire (pts (xy 370.84 45.72) (xy 367.03 45.72))
+    (stroke (width 0) (type default) (color 0 0 0 0))
+  )
   (bus (pts (xy 17.78 133.35) (xy 17.78 135.89))
     (stroke (width 0) (type default) (color 0 0 0 0))
@@
     (stroke (width 0) (type default) (color 0 0 0 0))
   )
+  (wire (pts (xy 280.67 124.46) (xy 280.67 123.19))
+    (stroke (width 0) (type default) (color 0 0 0 0))
+  )
   (wire (pts (xy 270.51 127) (xy 284.48 127))
     (stroke (width 0) (type default) (color 0 0 0 0))
@@
     (stroke (width 0) (type default) (color 0 0 0 0))
   )
-  (wire (pts (xy 381 116.84) (xy 378.46 116.84))
-    (stroke (width 0) (type default) (color 0 0 0 0))
-  )
   (polyline (pts (xy 15.24 17.78) (xy 15.24 107.95))
     (stroke (width 0) (type default) (color 0 0 0 0))
@@
     (stroke (width 0) (type default) (color 0 0 0 0))
   )
-  (wire (pts (xy 370.84 43.18) (xy 367.03 43.18))
-    (stroke (width 0) (type default) (color 0 0 0 0))
-  )
   (polyline (pts (xy 401.32 33.02) (xy 401.32 105.41))
     (stroke (width 0) (type default) (color 0 0 0 0))
@@
     (stroke (width 0) (type default) (color 0 0 0 0))
   )
-  (wire (pts (xy 378.46 121.92) (xy 378.46 116.84))
-    (stroke (width 0) (type default) (color 0 0 0 0))
-  )
   (wire (pts (xy 86.36 86.36) (xy 86.36 100.33))
     (stroke (width 0) (type default) (color 0 0 0 0))
@@
     (stroke (width 0) (type default) (color 0 0 0 0))
   )
-  (wire (pts (xy 370.84 40.64) (xy 370.84 43.18))
+  (wire (pts (xy 370.84 40.64) (xy 370.84 45.72))
     (stroke (width 0) (type default) (color 0 0 0 0))
   )
@@
     (stroke (width 0) (type default) (color 0 0 0 0))
   )
-  (wire (pts (xy 280.67 123.19) (xy 280.67 121.92))
-    (stroke (width 0) (type default) (color 0 0 0 0))
-  )
-  (wire (pts (xy 280.67 121.92) (xy 280.67 116.84))
+  (wire (pts (xy 280.67 116.84) (xy 280.67 123.19))
     (stroke (width 0) (type default) (color 0 0 0 0))
   )
@@
     (stroke (width 0) (type default) (color 0 0 0 0))
   )
+  (wire (pts (xy 270.51 124.46) (xy 280.67 124.46))
+    (stroke (width 0) (type default) (color 0 0 0 0))
+  )
   (wire (pts (xy 109.22 163.83) (xy 121.92 163.83))
     (stroke (width 0) (type default) (color 0 0 0 0))
@@
     (stroke (width 0) (type default) (color 0 0 0 0))
   )
-  (image (at 392.43 237.49) (scale 0.749531)
+  (image (at 375.92 220.98) (scale 1.49758)
     (data
       iVBORw0KGgoAAAANSUhEUgAAAfQAAAH0CAYAAADL1t+KAAAABHNCSVQICAgIfAhkiAAAAAlwSFlz
@@
     (pin "2")
   )
-  (symbol (lib_id "power:VBUS") (at 381 116.84 270) (unit 1)
+  (symbol (lib_id "power:VBUS") (at 368.3 124.46 270) (unit 1)
     (in_bom yes) (on_board yes) (fields_autoplaced)
-    (property "Reference" "#PWR025" (id 0) (at 377.19 116.84 0)
+    (property "Reference" "#PWR025" (id 0) (at 364.49 124.46 0)
       (effects (font (size 1.27 1.27)) hide)
     )
-    (property "Value" "VBUS" (id 1) (at 384.81 116.8399 90)
+    (property "Value" "VBUS" (id 1) (at 372.11 124.4599 90)
       (effects (font (size 1.27 1.27)) (justify left))
     )
-    (property "Footprint" "" (id 2) (at 381 116.84 0)
+    (property "Footprint" "" (id 2) (at 368.3 124.46 0)
       (effects (font (size 1.27 1.27)) hide)
     )
-    (property "Datasheet" "" (id 3) (at 381 116.84 0)
+    (property "Datasheet" "" (id 3) (at 368.3 124.46 0)
       (effects (font (size 1.27 1.27)) hide)
     )

Commit message: feat: final viper board changes
Signed-off-by: Matt Gleich <git@mattglei.ch>
Parts:
- J11: value Conn_01x05_Male -> Adafruit Quad Alphanumeric I2C Backpack
Connections:
- net GND: now also J11.3 (Pin_3), J15.6 (Pin_6), U1.38 (GND), U2.38 (GND), U4.38 (GND); no longer U1.3 (GND), U2.3 (GND), U4.3 (GND)
- no-connect marks 382 -> 384
Changed lines of the file:
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@@
   (junction (at 81.28 57.15) (diameter 0) (color 0 0 0 0)
   )
+  (junction (at 369.57 48.26) (diameter 0) (color 0 0 0 0)
+  )
   (junction (at 88.9 35.56) (diameter 0) (color 0 0 0 0)
   )
@@
   (junction (at 280.67 123.19) (diameter 0) (color 0 0 0 0)
   )
+  (junction (at 273.05 127) (diameter 0) (color 0 0 0 0)
+  )
   (no_connect (at 121.92 248.92))
   (no_connect (at 45.72 259.08))
+  (no_connect (at 331.47 48.26))
   (no_connect (at 90.17 246.38))
   (no_connect (at 166.37 171.45))
@@
   (no_connect (at 166.37 146.05))
   (no_connect (at 392.43 74.93))
+  (no_connect (at 332.74 127))
   (no_connect (at 392.43 69.85))
   (no_connect (at 166.37 179.07))
@@
   (no_connect (at 33.02 161.29))
   (no_connect (at 368.3 137.16))
-  (no_connect (at 368.3 127))
   (no_connect (at 90.17 236.22))
   (no_connect (at 179.07 184.15))
@@
   (no_connect (at 379.73 74.93))
   (no_connect (at 367.03 81.28))
+  (no_connect (at 234.95 127))
   (no_connect (at 368.3 157.48))
   (no_connect (at 166.37 166.37))
@@
     (stroke (width 0) (type default) (color 0 0 0 0))
   )
-  (wire (pts (xy 367.03 48.26) (xy 372.11 48.26))
+  (wire (pts (xy 367.03 48.26) (xy 369.57 48.26))
     (stroke (width 0) (type default) (color 0 0 0 0))
   )
@@
     (stroke (width 0) (type default) (color 0 0 0 0))
   )
+  (wire (pts (xy 369.57 35.56) (xy 369.57 48.26))
+    (stroke (width 0) (type default) (color 0 0 0 0))
+  )
   (bus (pts (xy 17.78 156.21) (xy 17.78 161.29))
     (stroke (width 0) (type default) (color 0 0 0 0))
@@
     (stroke (width 0) (type default) (color 0 0 0 0))
   )
-  (wire (pts (xy 270.51 127) (xy 284.48 127))
+  (wire (pts (xy 270.51 127) (xy 273.05 127))
     (stroke (width 0) (type default) (color 0 0 0 0))
   )
@@
     (stroke (width 0) (type default) (color 0 0 0 0))
   )
+  (wire (pts (xy 273.05 114.3) (xy 273.05 127))
+    (stroke (width 0) (type default) (color 0 0 0 0))
+  )
   (wire (pts (xy 374.65 46.99) (xy 374.65 88.9))
     (stroke (width 0) (type default) (color 0 0 0 0))
@@
     (stroke (width 0) (type default) (color 0 0 0 0))
   )
+  (wire (pts (xy 273.05 127) (xy 284.48 127))
+    (stroke (width 0) (type default) (color 0 0 0 0))
+  )
   (wire (pts (xy 251.46 39.37) (xy 251.46 53.34))
     (stroke (width 0) (type default) (color 0 0 0 0))
@@
     (stroke (width 0) (type default) (color 0 0 0 0))
   )
+  (wire (pts (xy 283.21 114.3) (xy 273.05 114.3))
+    (stroke (width 0) (type default) (color 0 0 0 0))
+  )
   (wire (pts (xy 49.53 119.38) (xy 49.53 124.46))
     (stroke (width 0) (type default) (color 0 0 0 0))
@@
     (stroke (width 0) (type default) (color 0 0 0 0))
   )
+  (wire (pts (xy 373.38 35.56) (xy 369.57 35.56))
+    (stroke (width 0) (type default) (color 0 0 0 0))
+  )
   (wire (pts (xy 115.57 73.66) (xy 115.57 86.36))
     (stroke (width 0) (type default) (color 0 0 0 0))
@@
     (stroke (width 0) (type default) (color 0 0 0 0))
   )
+  (wire (pts (xy 369.57 48.26) (xy 372.11 48.26))
+    (stroke (width 0) (type default) (color 0 0 0 0))
+  )
   (wire (pts (xy 173.99 39.37) (xy 175.26 39.37))
     (stroke (width 0) (type default) (color 0 0 0 0))
@@
     (pin "2")
   )
+  (symbol (lib_id "power:GND") (at 373.38 35.56 90) (unit 1)
+    (in_bom yes) (on_board yes) (fields_autoplaced)
+    (property "Reference" "#PWR0107" (id 0) (at 379.73 35.56 0)
+      (effects (font (size 1.27 1.27)) hide)
+    )
+    (property "Value" "GND" (id 1) (at 377.19 35.5599 90)
+      (effects (font (size 1.27 1.27)) (justify right))
+    )
+    (property "Footprint" "" (id 2) (at 373.38 35.56 0)
+      (effects (font (size 1.27 1.27)) hide)
+    )
+    (property "Datasheet" "" (id 3) (at 373.38 35.56 0)
+      (effects (font (size 1.27 1.27)) hide)
+    )
+    (pin "1")
+  )
   (symbol (lib_id "power:GND") (at 218.44 167.64 90) (unit 1)
     (in_bom yes) (on_board yes) (fields_autoplaced)
@@
     (pin "9")
   )
+  (symbol (lib_id "power:GND") (at 283.21 114.3 90) (unit 1)
+    (in_bom yes) (on_board yes) (fields_autoplaced)
+    (property "Reference" "#PWR?" (id 0) (at 289.56 114.3 0)
+      (effects (font (size 1.27 1.27)) hide)
+    )
+    (property "Value" "GND" (id 1) (at 287.02 114.2999 90)
+      (effects (font (size 1.27 1.27)) (justify right))
+    )
+    (property "Footprint" "" (id 2) (at 283.21 114.3 0)
+      (effects (font (size 1.27 1.27)) hide)
+    )
+    (property "Datasheet" "" (id 3) (at 283.21 114.3 0)
+      (effects (font (size 1.27 1.27)) hide)
+    )
+    (pin "1")
+  )
   (symbol (lib_id "Device:LED") (at 143.51 86.36 0) (unit 1)
     (in_bom yes) (on_board yes) (fields_autoplaced)
@@
     (pin "2")
   )
-  (symbol (lib_id "power:GND") (at 234.95 127 270) (unit 1)
-    (in_bom yes) (on_board yes) (fields_autoplaced)
-    (property "Reference" "#PWR0111" (id 0) (at 228.6 127 0)
-      (effects (font (size 1.27 1.27)) hide)
-    )
-    (property "Value" "GND" (id 1) (at 231.14 126.9999 90)
-      (effects (font (size 1.27 1.27)) (justify right))
-    )
-    (property "Footprint" "" (id 2) (at 234.95 127 0)
-      (effects (font (size 1.27 1.27)) hide)
-    )
-    (property "Datasheet" "" (id 3) (at 234.95 127 0)
-      (effects (font (size 1.27 1.27)) hide)
-    )
-    (pin "1")
-  )
   (symbol (lib_id "power:VBUS") (at 68.58 45.72 270) (unit 1)
     (in_bom yes) (on_board yes) (fields_autoplaced)
@@
       (effects (font (size 1.27 1.27)) (justify right))
     )
-    (property "Value" "Conn_01x05_Male" (id 1) (at 276.86 137.16 0)
+    (property "Value" "Adafruit Quad Alphanumeric I2C Backpack" (id 1) (at 292.1 162.56 90)
       (effects (font (size 1.27 1.27)) (justify right))
     )
@@
     (pin "2")
   )
-  (symbol (lib_id "power:GND") (at 332.74 127 270) (unit 1)
-    (in_bom yes) (on_board yes) (fields_autoplaced)
-    (property "Reference" "#PWR023" (id 0) (at 326.39 127 0)
-      (effects (font (size 1.27 1.27)) hide)
-    )
-    (property "Value" "GND" (id 1) (at 328.93 126.9999 90)
-      (effects (font (size 1.27 1.27)) (justify right))
-    )
-    (property "Footprint" "" (id 2) (at 332.74 127 0)
-      (effects (font (size 1.27 1.27)) hide)
-    )
-    (property "Datasheet" "" (id 3) (at 332.74 127 0)
-      (effects (font (size 1.27 1.27)) hide)
-    )
-    (pin "1")
-  )
   (symbol (lib_id "Device:LED") (at 93.98 86.36 0) (unit 1)
     (in_bom yes) (on_board yes) (fields_autoplaced)
@@
     (pin "2")
   )
-  (symbol (lib_id "power:GND") (at 331.47 48.26 270) (unit 1)
-    (in_bom yes) (on_board yes) (fields_autoplaced)
-    (property "Reference" "#PWR0117" (id 0) (at 325.12 48.26 0)
-      (effects (font (size 1.27 1.27)) hide)
-    )
-    (property "Value" "GND" (id 1) (at 327.66 48.2599 90)
-      (effects (font (size 1.27 1.27)) (justify right))
-    )
-    (property "Footprint" "" (id 2) (at 331.47 48.26 0)
-      (effects (font (size 1.27 1.27)) hide)
-    )
-    (property "Datasheet" "" (id 3) (at 331.47 48.26 0)
-      (effects (font (size 1.27 1.27)) hide)
-    )
-    (pin "1")
-  )
   (symbol (lib_id "Device:R_US") (at 204.47 39.37 90) (unit 1)
     (in_bom yes) (on_board yes) (fields_autoplaced)
@@
     (pin "1")
   )
+  (symbol (lib_id "power:GND") (at 368.3 127 90) (unit 1)
+    (in_bom yes) (on_board yes) (fields_autoplaced)
+    (property "Reference" "#PWR?" (id 0) (at 374.65 127 0)
+      (effects (font (size 1.27 1.27)) hide)
+    )
+    (property "Value" "GND" (id 1) (at 372.11 126.9999 90)
+      (effects (font (size 1.27 1.27)) (justify right))
+    )
+    (property "Footprint" "" (id 2) (at 368.3 127 0)
+      (effects (font (size 1.27 1.27)) hide)
+    )
+    (property "Datasheet" "" (id 3) (at 368.3 127 0)
+      (effects (font (size 1.27 1.27)) hide)
+    )
+    (pin "1")
+  )
   (symbol (lib_id "power:GND") (at 350.52 175.26 0) (unit 1)
     (in_bom yes) (on_board yes) (fields_autoplaced)
@@
       (reference "#PWR018") (unit 1) (value "GND") (footprint "")
     )
-    (path "/cc313d92-56e1-4eab-bd63-f2ea29091004"
-      (reference "#PWR023") (unit 1) (value "GND") (footprint "")
-    )
     (path "/ebde721f-8375-4826-b32e-f21c8748d713"
       (reference "#PWR024") (unit 1) (value "GND") (footprint "")
@@
       (reference "#PWR0106") (unit 1) (value "GND") (footprint "")
     )
+    (path "/3bfcf9a4-0609-42ba-a923-60777e5cc65f"
+      (reference "#PWR0107") (unit 1) (value "GND") (footprint "")
+    )
     (path "/08aa315e-6f02-44a8-8152-f1d4497ecc9a"
       (reference "#PWR0108") (unit 1) (value "GND") (footprint "")
@@
       (reference "#PWR0110") (unit 1) (value "VBUS") (footprint "")
     )
-    (path "/7e9bb2b4-4718-4b7a-89b2-88a429383acd"
-      (reference "#PWR0111") (unit 1) (value "GND") (footprint "")
-    )
     (path "/3e60494b-aa6e-45bf-8f72-ae3dce78ba8e"
       (reference "#PWR0113") (unit 1) (value "GND") (footprint "")
@@
       (reference "#PWR0116") (unit 1) (value "VBUS") (footprint "")
     )
-    (path "/d3594629-d674-4742-af99-c21a97acf6f5"
-      (reference "#PWR0117") (unit 1) (value "GND") (footprint "")
-    )
     (path "/86a43539-fdb5-42b1-bdcc-be42c9608e44"
       (reference "#PWR0122") (unit 1) (value "GND") (footprint "")
@@
       (reference "#PWR0127") (unit 1) (value "VBUS") (footprint "")
     )
+    (path "/69440381-319f-4ee1-afba-40ce3ef26e88"
+      (reference "#PWR?") (unit 1) (value "GND") (footprint "")
+    )
+    (path "/e5b7c2e0-9f05-43c4-b5a4-35c25b33d437"
+      (reference "#PWR?") (unit 1) (value "GND") (footprint "")
+    )
     (path "/3ba435c3-0cd1-440e-b45b-f254734fef9c"
       (reference "Brd1") (unit 1) (value "SSD1306") (footprint "SSD1306:128x64OLED")
@@
     )
     (path "/8a1cab7c-8bac-408e-8651-e6543692bd62"
-      (reference "J11") (unit 1) (value "Conn_01x05_Male") (footprint "Connector_PinHeader_2.54mm:PinHeader_1x05_P2.54mm_Vertical")
+      (reference "J11") (unit 1) (value "Adafruit Quad Alphanumeric I2C Backpack") (footprint "Connector_PinHeader_2.54mm:PinHeader_1x05_P2.54mm_Vertical")
     )
     (path "/b6241319-1409-4552-bb2a-fd457a961a4d"
